File: hardware/epaper-display.kicad_sch (KiCad schematic)
At the start: 72 parts, among them J1 AES200200A00 FPC, J2 USB-C 2.0 receptacle, J3 LiPo cell (B+/B-), J4 I2C temp (optional), J5 UART, J6 GPIO expansion, Q1 Si1304BDL / NX3008NBK, Q2 FS8205A, SW1 EN/RESET, SW2 BOOT, SW3 BTN_UP, SW4 BTN_DOWN, SW5 BTN_LEFT, SW6 BTN_RIGHT, SW7 BTN_SELECT, SW8 BTN_CANCEL, U1 ESP32-S3-WROOM-1-N8, U2 MCP73831T-2ACI/OT, U3 TLV75733PDBVR, U4 DW01A

Commit message: hardware: correct Q2 FS8205A pinout to the Tech Public drawing
The FS8205A pinout is resolved, and the mapping previously wired was
wrong. Corrected to what the "Package and Pin Configuration" drawing in
components/fs8205a-techpublic.pdf shows:

    pin 6  G1      pin 5  D1/D2      pin 4  G2
    pin 1  S1      pin 2  D1/D2      pin 3  S2

Each FET half occupies one END of the package (FET1 = S1/G1 on pins 1/6,
FET2 = S2/G2 on pins 3/4) with the common drain on the two MIDDLE pins.
A symmetric leadframe, which is corroborating in itself.

This is NOT the commonly-quoted 8205A mapping (1=S1 2=G1 3=S2 4=G2 5=D2
6=D1) that the previous revision used, and the difference mattered: pins
2 and 6 were swapped between gate and drain, so PROT_DO was driven into
a drain and G1 was tied to the drain node. The DW01A could not have held
either FET off and the protection would have silently done nothing --
the worst failure mode available to a safety circuit, since the board
would have looked and behaved fine right up until it over-discharged the
cell.

Netlist now:

    Q2.1 S1 = BATT_NEG   Q2.6 G1 = PROT_DO  (discharge, source B-)
    Q2.3 S2 = GND        Q2.4 G2 = PROT_CO  (charge, source P-)
    Q2.2 / Q2.5 D1/D2 = PROT_MID

verified against the DW01A's drive convention: it turns the discharge
FET off by pulling DO to VSS and the charge FET off by pulling CO to VM,
so each gate must reference the source at its own end.

The warnings that said "unresolved, measure before ordering a PCB" are
replaced with a note that the pinout is unusual and that pin assignments
must NOT be copied from other 8205A designs. A DMM confirmation is still
suggested because it costs nothing, but it is no longer a blocker.

Also drops a stale status bullet that still described the MCP1825S's
120 uA quiescent current as the design's open item; that was fixed when
U3 became the TLV75733P.

Co-Authored-By: Claude Opus 5 <noreply@anthropic.com>
Claude-Session: https://claude.ai/code/session_017ASByNz7rVoZ3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
Connections:
- net PROT_DO: now also Q2.6 (G1); no longer Q2.2 (G1)
- net PROT_MID: now also Q2.2 (D1/D2); no longer Q2.6 (D1)
Other:
- note added: "Q2 pinout is 1=S1 2=D 3=S2 4=G2 5=D 6=G1, per the Package and Pin Configuration"
- note added: "commonly-quoted 8205A mapping (2=G1, 6=D1) - do not copy that from other"
- note added: "designs. Confirm once with a DMM: shorted pair = drains, ~0.6V in diode mode"
- note added: "drawing in components/fs8205a-techpublic.pdf. Each FET half sits at one END of"
- note added: "the package and the common drain is on the two MIDDLE pins. This is NOT the"
- note added: "to the drain node = a source, remaining two = gates."
- note removed: "*** Q2 PIN NUMBERING IS UNRESOLVED - MEASURE BEFORE ORDERING A PCB ***"
- note removed: "DMM check: shorted pair = drains; diode-mode ~0.6V to the drain node = a"
- note removed: "Neither FS8205A datasheet in components/ gives a pin-number table. The Tech"
- note removed: "Public drawing shows rows S1/D/S2 and G1/D/G2, which CONTRADICTS the mapping"
- note removed: "source; the remaining two are gates. See README section 4."
- note removed: "wired here (1=S1 2=G1 3=S2 4=G2 5=D2 6=D1). Candidate B is 2=D and 6=G1."

Commit message: hardware: fix J2 shield pad name, connect J1 hold-downs, make UUIDs stable
Four fixes, all surfaced while bringing up the PCB from this schematic.

J2 shield pin was numbered S1, but every USB-C footprint in KiCad's
Connector_USB library names its shield pads SH -- S1 is what KiCad's own
USB-C *symbol* uses.  "Update PCB from Schematic" failed outright with
"pad S1 not found in Connector_USB:USB_C_Receptacle_GCT_USB4085".

J1's Hirose FH12 footprint has two mechanical hold-down tabs (both pads
named MP) with no matching symbol pin, so they were left floating -- a
silent mismatch, since KiCad does not flag unmatched footprint pads.
Added an MP pin tied to GND; those tabs are what hold the connector down
against FPC insertion force.

UUIDs were uuid4(), regenerated on every run.  KiCad links each footprint
to its schematic symbol by the symbol's UUID, so re-running this script
after starting a layout would orphan every footprint on the board.  They
are now uuid5 hashes of stable keys (sym:<ref>, pin:<ref>:<num>, ...),
and U() raises on a duplicate key.  Output is byte-identical across runs,
so the git diff also stays empty when nothing actually changed.

Cleared the three remaining ERC errors, all spurious: J1 VPP is the
panel's OTP programming pin rather than a supply rail, so it is passive,
not power_in; PROT_VDD and BATT_NEG are sourced from the cell through
J3, a passive connector pin that ERC cannot see as a driver, so they get
PWR_FLAGs like VBUS and GND already had.

Verified with kicad-cli 10.0.3: ERC 0 errors 0 warnings, netlist exports
clean with 72 components and every footprint assigned.  epaper-display
.kicad_pro also picks up KiCad 10's expansion of its default settings
from the project having been opened in the GUI.

Co-Authored-By: Claude Opus 5 (1M context) <noreply@anthropic.com>
Connections:
- net GND: now also J1.MP, J2.SH (SHIELD); no longer J2.S1 (SHIELD)

Commit message: hardware: reorganise J6 into a blocked SPI/I2C/ADC expansion header
J6 was a 2x12 that broke 15 spare GPIOs out in numeric order and padded
the last six positions with GND. Same 15 GPIOs now sit on a 2x10 laid out
in functional blocks, so a peripheral wires to one contiguous corner:

  1-8   3V3, GND, SPI SCLK/MOSI/MISO/CS (IO38-41), IRQ (IO11), GND
  9-10  I2C SDA/SCL (IO12/IO13), R26/R27 4.7k pull-ups fitted DNP
  11,13 ADC1 inputs (IO2, IO10), each facing a GND pin
  15-20 six spare GPIOs, with the PSRAM-variant-sensitive ones last

Two choices drove the pin picks:

* The IRQ line is an RTC GPIO. Only GPIO0-21 can wake the chip from deep
  sleep through EXT1, so an interrupt on GPIO35-48 could not wake a board
  that is asleep 99.98 % of the time.
* ADC1 is the only ADC usable while Wi-Fi is running, and it exists only
  on GPIO1-10 -- of which GPIO1 is VBAT_SENSE, GPIO3 is the JTAG strap and
  GPIO4-9 are the panel. GPIO2 and GPIO10 were therefore the board's last
  two Wi-Fi-safe analog pins, and both were spent on push buttons.

So the six user buttons move from GPIO2/GPIO10-13 to GPIO14-18/GPIO21.
All six replacements are still RTC GPIOs, so every button remains an EXT1
wake source; a button does not care which pin it sits on, an ADC input
does. Vacating GPIO11/12/13 also leaves the FSPID/FSPICLK/FSPIQ IO MUX
trio on the header for firmware that needs a true 80 MHz SPI2 bus.

Firmware written against the old button map is stale -- see README 7.

Co-Authored-By: Claude Opus 5 <noreply@anthropic.com>
Claude-Session: https://claude.ai/code/session_01SzeYyBp5QCecUgqrvxzkBP
Parts:
- added R26, R27: 4.7k (DNP), Resistor_SMD:R_0805_2012Metric, symbol epaper:R
- J6: footprint Connector_PinHeader_2.54mm:PinHeader_2x12_P2.54mm_Vertical -> Connector_PinHeader_2.54mm:PinHeader_2x10_P2.54mm_Vertical; symbol epaper:Conn_2x12 -> epaper:Conn_2x10
Connections:
- net +3V3: now also R26.1, R27.1
- net BTN_CANCEL: now also U1.23 (IO21); no longer U1.22 (IO14)
- net BTN_DOWN: now also U1.8 (IO15); no longer U1.18 (IO10)
- net BTN_LEFT: now also U1.9 (IO16); no longer U1.19 (IO11)
- net BTN_RIGHT: now also U1.10 (IO17); no longer U1.20 (IO12)
- net BTN_SELECT: now also U1.11 (IO18); no longer U1.21 (IO13)
- net BTN_UP: now also U1.22 (IO14); no longer U1.38 (IO2)
- net EXP_IO35: now also J6.18; no longer J6.8
- net EXP_IO36: now also J6.19; no longer J6.9
- net EXP_IO37: now also J6.20; no longer J6.10
- net GND: now also J6.12, J6.14, J6.8; no longer J6.18, J6.19, J6.20, J6.21, J6.22, J6.23, J6.24
- net EXP_IO15 renamed EXP_SPI_SCLK
- net EXP_SPI_SCLK: now also U1.31 (IO38); no longer U1.8 (IO15)
- net EXP_IO16 renamed EXP_SPI_MOSI
- net EXP_SPI_MOSI: now also U1.32 (IO39); no longer U1.9 (IO16)
- net EXP_IO17 renamed EXP_SPI_MISO
- net EXP_SPI_MISO: now also U1.33 (IO40); no longer U1.10 (IO17)
- net EXP_IO18 renamed EXP_SPI_CS
- net EXP_SPI_CS: now also U1.34 (IO41); no longer U1.11 (IO18)
- net EXP_IO21 renamed EXP_IRQ
- net EXP_IRQ: now also U1.19 (IO11); no longer U1.23 (IO21)
- net EXP_IO38 renamed EXP_ADC_A
- net EXP_ADC_A: now also U1.38 (IO2); no longer U1.31 (IO38)
- removed net EXP_IO39: J6.12, U1.32 (IO39)
- net EXP_IO40 renamed EXP_ADC_B
- net EXP_ADC_B: now also U1.18 (IO10); no longer U1.33 (IO40)
- removed net EXP_IO41: J6.14, U1.34 (IO41)
- new net EXP_SCL: J6.10, R27.2, U1.21 (IO13)
- new net EXP_SDA: J6.9, R26.2, U1.20 (IO12)
Other:
- note added: "(IO2/IO10, the only ADC pins usable with Wi-Fi on); 15-20 = spares."
- note added: "1-8 = 3V3/GND + SPI SCLK,MOSI,MISO,CS (IO38-41) + IRQ (IO11) + GND;"
- note added: "9/10 = I2C SDA/SCL (IO12/13, R26/R27 pull-ups DNP); 11/13 = ADC1 in"
- note added: "IO35-37 (pins 18-20) and IO47/48 (16/17) assume a non-octal-PSRAM,"
- note added: "J6 (2x10 expansion) is laid out in blocks, NOT in GPIO order:"
- note added: "non-R16VA module. Buttons moved to IO14-18/IO21 to free IO2/IO10-13."
- note removed: "J6 IO35-37 and IO47/48 assume non-octal-PSRAM, non-R16V module"

Commit message: hardware: switch the main processor to ESP32-C6-WROOM-1-N8 (RISC-V)
Replaces the ESP32-S3-WROOM-1-N8 (dual-core Xtensa) with the
ESP32-C6-WROOM-1-N8 (single-core RISC-V, Wi-Fi 6 / BLE 5.3 / 802.15.4).
Same 18.0 x 25.5 x 3.1 mm module outline, but 29 pads against 41 in a
different order, so this is a full symbol, footprint and pin-map change --
not a drop-in. All pin data is taken from Table 3-1 and chapter 4 of
components/esp32-c6-wroom-1_wroom-1u_datasheet_en.pdf (v1.4).

The C6 breaks out 23 usable GPIOs where the S3 gave 36, and three scarce
resources share the same GPIO0-GPIO7 block: LP (RTC) IOs, which are the
only pins EXT1 can wake from; ADC1, the chip's only ADC; and the SPI2 IO
MUX pins. Six wake-capable buttons plus battery sense claim seven of the
eight LP pins, which forces the rest of the allocation:

  * buttons  -> GPIO2-GPIO7 (GPIO7 takes one because it is the only LP
    pin with no ADC channel, so spending it on a button wastes nothing)
  * VBAT_SENSE -> GPIO0 (ADC1_CH0); the one LP pin left, GPIO1, is both
    ADC1_CH1 and LP_GPIO1 and goes to the expansion header
  * panel     -> GPIO18-GPIO23, via the GPIO matrix rather than the SPI2
    IO MUX (every IO MUX pin is a button or UART0); 40 MHz there is far
    above what an SSD1681 needs
  * USB       -> GPIO12/GPIO13, fixed by the USB Serial/JTAG PHY
  * UART0     -> GPIO16/GPIO17; BOOT -> GPIO9

Strapping changes: R15 becomes a 10k pull-UP on GPIO15, not a pull-down.
Datasheet Table 4-7 makes GPIO15 = 1 keep JTAG on the USB Serial/JTAG
controller once EFUSE_JTAG_SEL_ENABLE is burnt, and GPIO15 = 0 move it to
the MTDI/MTCK/MTMS/MTDO pads -- which are GPIO4-GPIO7, i.e. four of the
buttons, so pad-JTAG is unreachable on this board. New R28 (10k pull-up)
holds GPIO8 high: joint download boot needs GPIO8 = 1 with GPIO9 = 0, and
GPIO8 = 0 with GPIO9 = 0 is an invalid combination.

J6 shrinks from 2x10 (15 GPIOs) to 2x4 (4 GPIOs): I2C pair on GPIO10/11,
one ADC-and-wake pin on GPIO1, one strap-constrai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
Parts:
- added R28: 10k, Resistor_SMD:R_0805_2012Metric, symbol epaper:R
- J6: footprint Connector_PinHeader_2.54mm:PinHeader_2x10_P2.54mm_Vertical -> Connector_PinHeader_2.54mm:PinHeader_2x04_P2.54mm_Vertical; symbol epaper:Conn_2x10 -> epaper:Conn_2x04
- U1: value ESP32-S3-WROOM-1-N8 -> ESP32-C6-WROOM-1-N8; footprint RF_Module:ESP32-S3-WROOM-1 -> Espressif:ESP32-C6-WROOM-1; symbol epaper:ESP32-S3-WROOM-1 -> epaper:ESP32-C6-WROOM-1
Connections:
- net +3V3: now also R15.1, R28.1
- net BOOT: now also U1.15 (IO9); no longer U1.27 (IO0)
- net BTN_CANCEL: now also U1.27 (IO2); no longer U1.23 (IO21)
- net BTN_DOWN: now also U1.5 (IO5); no longer U1.8 (IO15)
- net BTN_LEFT: now also U1.6 (IO6); no longer U1.9 (IO16)
- net BTN_RIGHT: now also U1.7 (IO7); no longer U1.10 (IO17)
- net BTN_SELECT: now also U1.26 (IO3); no longer U1.11 (IO18)
- net BTN_UP: now also U1.4 (IO4); no longer U1.22 (IO14)
- net EPD_BUSY: now also U1.16 (IO18); no longer U1.17 (IO9)
- net EPD_CS: now also U1.19 (IO21); no longer U1.6 (IO6)
- net EPD_DC: now also U1.18 (IO20); no longer U1.7 (IO7)
- net EPD_MOSI: now also U1.20 (IO22); no longer U1.5 (IO5)
- net EPD_RST: now also U1.17 (IO19); no longer U1.12 (IO8)
- net EPD_SCLK: now also U1.21 (IO23); no longer U1.4 (IO4)
- net EXP_SCL: now also J6.4, U1.12 (IO11); no longer J6.10, U1.21 (IO13)
- net EXP_SDA: now also J6.3, U1.11 (IO10); no longer J6.9, U1.20 (IO12)
- net GND: now also J6.6, U1.28 (GND), U1.29 (EPAD); no longer J6.12, J6.14, R15.2, U1.40 (GND), U1.41 (EPAD)
- net UART_RXD0: now also U1.24 (RXD0); no longer U1.36 (RXD0)
- net UART_TXD0: now also U1.25 (TXD0); no longer U1.37 (TXD0)
- net VBAT_SENSE: now also U1.8 (IO0); no longer U1.39 (IO1)
- removed net EXP_ADC_A: J6.11, U1.38 (IO2)
- removed net EXP_ADC_B: J6.13, U1.18 (IO10)
- removed net EXP_IO35: J6.18, U1.28 (IO35)
- removed net EXP_IO36: J6.19, U1.29 (IO36)
- removed net EXP_IO37: J6.20, U1.30 (IO37)
- removed net EXP_IO42: J6.15, U1.35 (IO42)
- removed net EXP_IO47: J6.16, U1.24 (IO47)
- removed net EXP_IO48: J6.17, U1.25 (IO48)
- net EXP_IRQ renamed EXP_IO8
- net EXP_IO8: now also U1.10 (IO8), R28.2; no longer U1.19 (IO11)
- removed net EXP_SPI_CS: J6.6, U1.34 (IO41)
- net EXP_SPI_MISO renamed EXP_ADC_IRQ
- net EXP_ADC_IRQ: now also U1.9 (IO1); no longer U1.33 (IO40)
- removed net EXP_SPI_MOSI: J6.4, U1.32 (IO39)
- removed net EXP_SPI_SCLK: J6.3, U1.31 (IO38)
- removed net STRAP_IO3: R15.1, U1.15 (IO3)
- new net STRAP_IO15: R15.2, U1.23 (IO15)
- no-connect marks 4 -> 2
Other:
- note added: "All six buttons sit on IO2-IO7 because the C6's LP (RTC) IOs are IO0-IO7 and"
- note added: "J6 (2x4 expansion) is 1=3V3 2=GND, 3/4=I2C SDA/SCL (IO10/IO11, R26/R27"
- note added: "J6 pin 7 is IO8, a STRAPPING pin held high by R28. Do not let anything"
- note added: "NOT draw a sustained 500mA from +3V3 via J6."
- note added: "R15 pulls IO15 HIGH (the S3 revision pulled its strap low). IO15 selects"
- note added: "RF_Module library has no C6-WROOM-1 - it only carries ESP32-C6-MINI-1."
- note added: "SW3/SW4 sit on MTMS/MTDI, which are also SDIO-slave clock-edge straps. R17/R18"
- note added: "Serial/JTAG, low = the MTMS/MTDI/MTCK/MTDO pads - which are IO4-IO7,"
- note added: "There is no SPI block: SPI2's IO MUX pins on the C6 (IO2/4/5/6/7/16)"
- note added: "U1 footprint is Espressif:ESP32-C6-WROOM-1, from Espressif's official KiCad"
- note added: "VBAT_SENSE (ADC1_CH0), IO1 goes to J6, and that is the whole LP budget."
- note added: "are all buttons or UART0 here. Four spare GPIOs is all the part has."
- note added: "burst load (C6 Wi-Fi TX peaks at 382mA, module datasheet Table 6-4), but do"
- note added: "i.e. four of the buttons. Required, not optional: IO15 has no internal"
- note added: "invalid boot mode) or the board stops being flashable over USB."
- note added: "latch them high at reset; this board never uses SDIO slave, so it is inert."
- note added: "library (install via KiCad's Plugin and Content Manager). Stock KiCad's"
- note added: "nothing else - only those eight pins can wake the chip through EXT1. IO0 is"
- note added: "pin that is both analog and EXT1-wake capable), 6/8=GND, 7=IO8 spare."
- note added: "plugged into J6 drive it low through reset (IO8=0 with IO9=0 is an"
- note added: "pull and must not float (module datasheet 4.4)."
- note added: "pull-ups DNP), 5=ADC/IRQ (IO1 = ADC1_CH1 AND LP_GPIO1 - the only spare"
- note added: "the JTAG source once EFUSE_JTAG_SEL_ENABLE is burnt: high = USB"
- note added: "through deep sleep; firmware may still enable LP pull-ups harmlessly in parallel."
- note removed: "(IO2/IO10, the only ADC pins usable with Wi-Fi on); 15-20 = spares."
- note removed: "1-8 = 3V3/GND + SPI SCLK,MOSI,MISO,CS (IO38-41) + IRQ (IO11) + GND;"
- note removed: "9/10 = I2C SDA/SCL (IO12/13, R26/R27 pull-ups DNP); 11/13 = ADC1 in"
- note removed: "IO35-37 (pins 18-20) and IO47/48 (16/17) assume a non-octal-PSRAM,"
- note removed: "J6 (2x10 expansion) is laid out in blocks, NOT in GPIO order:"
- note removed: "burst load, but do NOT draw a sustained 500mA from +3V3 via J6."
- note removed: "non-R16VA module. Buttons moved to IO14-18/IO21 to free IO2/IO10-13."
- note removed: "through deep sleep; firmware may still enable RTC pull-ups harmlessly in parallel."
- moved on the sheet: R26, R27
